Commit message: editted spawner to spawn red/blue/yellow blocks and cylinders

File: urdf/blue_cylinder.urdf (robot description, URDF)
Before this commit: robot blue_cylinder, 1 links, 0 joints
Links:
- link base_link: mass 0.00001 -> 0.04; geometry collision cylinder length=0.025 radius=0.06; visual cylinder length=0.025 radius=0.06

File: urdf/red_cylinder.urdf (robot description, URDF)
Before this commit: robot red_cylinder, 1 links, 0 joints
Links:
- link base_link: mass 0.00001 -> 0.04; geometry collision cylinder length=0.025 radius=0.06; visual cylinder length=0.025 radius=0.06

File: urdf/yellow_cylinder.urdf (robot description, URDF)
Before this commit: robot yellow_cylinder, 1 links, 0 joints
Links:
- link base_link: mass 0.00001 -> 0.04; geometry collision cylinder length=0.025 radius=0.06; visual cylinder length=0.025 radius=0.06
